File: tools/ergogen/output/pcbs/keyboard.kicad_pcb (KiCad board)
At the start: 2 copper layers, 357 x 104.5 mm, 102 parts

Commit message: chore(devenv): server moved to process-compose, scripts kept for one-shots
devenv has full process management (process-compose under the hood) — use
`devenv up` to start the long-running webtool server, supervised with
auto-restart. One-shot commands stay as scripts: `devenv shell -- ergogen`
runs the static config build, `devenv shell -- render` renders the current
PCB to PNGs.

Removed standalone `dev` script (replaced by `processes.server`).
Parts:
- moved D20 172.1 mm to (338.0, -114.0)
- moved LED20 172.1 mm to (332.0, -122.9)
- moved S20 172.1 mm to (332.0, -118.0)
- moved D3 159.2 mm to (74.0, -114.0)
- moved LED3 159.2 mm to (80.0, -122.9)
- moved S3 159.2 mm to (80.0, -118.0)
- moved D32 155.7 mm to (262.0, -123.1)
- moved LED32 155.7 mm to (256.0, -132.1)
- moved S32 155.7 mm to (256.0, -127.1)
- moved D23 152.3 mm to (319.0, -125.0)
- moved D29 152.3 mm to (281.0, -125.0)
- moved LED23 152.3 mm to (313.0, -134.0)
- moved LED29 152.3 mm to (275.0, -134.0)
- moved S23 152.3 mm to (313.0, -129.0)
- moved S29 152.3 mm to (275.0, -129.0)
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Connections:
- net TROW0 renamed ROW3
- net c0_r0 renamed pinky_top
- net c0_r1 renamed pinky_home
- net c0_r2 renamed pinky_bot
- net c1_r0 renamed ring_top
- net c1_r1 renamed ring_home
- net c1_r2 renamed ring_bot
- net c2_r0 renamed middle_top
- net c2_r1 renamed middle_home
- net c2_r2 renamed middle_bot
- net c3_r0 renamed index_top
- net c3_r1 renamed index_home
- net c3_r2 renamed index_bot
- net c4_r0 renamed inner_top
- net c4_r1 renamed inner_home
- net c4_r2 renamed inner_bot
- net led_din_matrix_c0_r0 renamed led_dout_matrix_pinky_top
- net led_din_matrix_c0_r1 renamed led_dout_matrix_pinky_home
- net led_din_matrix_c0_r2 renamed led_dout_matrix_pinky_bot
- net led_din_matrix_c1_r0 renamed led_dout_matrix_ring_top
- net led_din_matrix_c1_r1 renamed led_dout_matrix_ring_home
- net led_din_matrix_c1_r2 renamed led_dout_matrix_ring_bot
- net led_din_matrix_c2_r0 renamed led_dout_matrix_middle_top
- net led_din_matrix_c2_r1 renamed led_dout_matrix_middle_home
- net led_din_matrix_c2_r2 renamed led_dout_matrix_middle_bot
- net led_din_matrix_c3_r0 renamed led_dout_matrix_index_top
- net led_din_matrix_c3_r1 renamed led_dout_matrix_index_home
- net led_din_matrix_c3_r2 renamed led_dout_matrix_index_bot
- net led_din_matrix_c4_r0 renamed led_dout_matrix_inner_top
- net led_din_matrix_c4_r1 renamed led_dout_matrix_inner_home
- net led_din_matrix_c4_r2 renamed led_dout_matrix_inner_bot
- net led_din_mirror_matrix_c0_r0 renamed led_dout_mirror_matrix_pinky_top
- net led_din_mirror_matrix_c0_r1 renamed led_dout_mirror_matrix_pinky_home
- net led_din_mirror_matrix_c0_r2 renamed led_dout_mirror_matrix_pinky_bot
- net led_din_mirror_matrix_c1_r0 renamed led_dout_mirror_matrix_ring_top
- net led_din_mirror_matrix_c1_r1 renamed led_dout_mirror_matrix_ring_home
- net led_din_mirror_matrix_c1_r2 renamed led_dout_mirror_matrix_ring_bot
- net led_din_mirror_matrix_c2_r0 renamed led_dout_mirror_matrix_middle_top
- net led_din_mirror_matrix_c2_r1 renamed led_dout_mirror_matrix_middle_home
- net led_din_mirror_matrix_c2_r2 renamed led_dout_mirror_matrix_middle_bot
- net led_din_mirror_matrix_c3_r0 renamed led_dout_mirror_matrix_index_top
- net led_din_mirror_matrix_c3_r1 renamed led_dout_mirror_matrix_index_home
- net led_din_mirror_matrix_c3_r2 renamed led_dout_mirror_matrix_index_bot
- net led_din_mirror_matrix_c4_r0 renamed led_dout_mirror_matrix_inner_top
- net led_din_mirror_matrix_c4_r1 renamed led_dout_mirror_matrix_inner_home
- net led_din_mirror_matrix_c4_r2 renamed led_dout_mirror_matrix_inner_bot
- net led_dout_matrix_c0_r0 renamed led_din_matrix_pinky_top
- net led_dout_matrix_c0_r1 renamed led_din_matrix_pinky_home
- net led_dout_matrix_c0_r2 renamed led_din_matrix_pinky_bot
- net led_dout_matrix_c1_r0 renamed led_din_matrix_ring_top
- net led_dout_matrix_c1_r1 renamed led_din_matrix_ring_home
- net led_dout_matrix_c1_r2 renamed led_din_matrix_ring_bot
- net led_dout_matrix_c2_r0 renamed led_din_matrix_middle_top
- net led_dout_matrix_c2_r1 renamed led_din_matrix_middle_home
- net led_dout_matrix_c2_r2 renamed led_din_matrix_middle_bot
- net led_dout_matrix_c3_r0 renamed led_din_matrix_index_top
- net led_dout_matrix_c3_r1 renamed led_din_matrix_index_home
- net led_dout_matrix_c3_r2 renamed led_din_matrix_index_bot
- net led_dout_matrix_c4_r0 renamed led_din_matrix_inner_top
- net led_dout_matrix_c4_r1 renamed led_din_matrix_inner_home
- net led_dout_matrix_c4_r2 renamed led_din_matrix_inner_bot
- net led_dout_mirror_matrix_c0_r0 renamed led_din_mirror_matrix_pinky_top
- net led_dout_mirror_matrix_c0_r1 renamed led_din_mirror_matrix_pinky_home
- net led_dout_mirror_matrix_c0_r2 renamed led_din_mirror_matrix_pinky_bot
- net led_dout_mirror_matrix_c1_r0 renamed led_din_mirror_matrix_ring_top
- net led_dout_mirror_matrix_c1_r1 renamed led_din_mirror_matrix_ring_home
- net led_dout_mirror_matrix_c1_r2 renamed led_din_mirror_matrix_ring_bot
- net led_dout_mirror_matrix_c2_r0 renamed led_din_mirror_matrix_middle_top
- net led_dout_mirror_matrix_c2_r1 renamed led_din_mirror_matrix_middle_home
- net led_dout_mirror_matrix_c2_r2 renamed led_din_mirror_matrix_middle_bot
- net led_dout_mirror_matrix_c3_r0 renamed led_din_mirror_matrix_index_top
- net led_dout_mirror_matrix_c3_r1 renamed led_din_mirror_matrix_index_home
- net led_dout_mirror_matrix_c3_r2 renamed led_din_mirror_matrix_index_bot
- net led_dout_mirror_matrix_c4_r0 renamed led_din_mirror_matrix_inner_top
- net led_dout_mirror_matrix_c4_r1 renamed led_din_mirror_matrix_inner_home
- net led_dout_mirror_matrix_c4_r2 renamed led_din_mirror_matrix_inner_bot
- net mirror_c0_r0 renamed mirror_pinky_top
- net mirror_c0_r1 renamed mirror_pinky_home
- net mirror_c0_r2 renamed mirror_pinky_bot
- net mirror_c1_r0 renamed mirror_ring_top
- net mirror_c1_r1 renamed mirror_ring_home
- net mirror_c1_r2 renamed mirror_ring_bot
- net mirror_c2_r0 renamed mirror_middle_top
- net mirror_c2_r1 renamed mirror_middle_home
- net mirror_c2_r2 renamed mirror_middle_bot
- net mirror_c3_r0 renamed mirror_index_top
- net mirror_c3_r1 renamed mirror_index_home
- net mirror_c3_r2 renamed mirror_index_bot
- net mirror_c4_r0 renamed mirror_inner_top
- net mirror_c4_r1 renamed mirror_inner_home
- net mirror_c4_r2 renamed mirror_inner_bot
- LED16 pad 2: led_dout_thumbs_t0_thumb -> led_din_thumbs_t0_thumb
- LED16 pad 4: led_din_thumbs_t0_thumb -> led_dout_thumbs_t0_thumb
- LED17 pad 2: led_dout_thumbs_t1_thumb -> led_din_thumbs_t1_thumb
- LED17 pad 4: led_din_thumbs_t1_thumb -> led_dout_thumbs_t1_thumb
- LED33 pad 2: led_dout_mirror_thumbs_t0_thumb -> led_din_mirror_thumbs_t0_thumb
- LED33 pad 4: led_din_mirror_thumbs_t0_thumb -> led_dout_mirror_thumbs_t0_thumb
- LED34 pad 2: led_dout_mirror_thumbs_t1_thumb -> led_din_mirror_thumbs_t1_thumb
- LED34 pad 4: led_din_mirror_thumbs_t1_thumb -> led_dout_mirror_thumbs_t1_thumb
- S16 pad 1: TCOL0 -> COL3
- S17 pad 1: TCOL1 -> COL4
- S33 pad 1: TCOL0 -> COL3
- S34 pad 1: TCOL1 -> COL4
Other:
- board size 357 x 104.5 mm -> 276 x 76.1 mm
