File: pcb/kicad/keyboard.kicad_pcb (KiCad board)
At the start: 2 copper layers, 22 x 22 mm, 3 parts

Commit message: feat(tools): webtool drives ergogen → KiCad → render pipeline
Major milestone: layout webtool now has a 'build PCB' button that
generates a KiCad PCB end-to-end from the atlas layout state.

Pipeline:
  webtool state → POST /api/build → server.mjs
    → layoutToErgogen() → ergogen YAML
    → ergogen.process() → KiCad 8 .kicad_pcb
    → kicad-cli render → top + bottom PNGs
    → webtool displays the PNG and build log

Files:
- tools/server.mjs              Express dev server (port 8000)
- tools/layout-to-ergogen.mjs   atlas-state → ergogen-YAML translator
- tools/ergogen/config.yaml     static reference config (full 34-key atlas)
- tools/ergogen/footprints/     ceoloide footprints (Choc, SK6812, SOD-123)
- tools/layout/index.html       webtool with new 'build PCB' button + render
                                preview tabs (top/bottom/yaml)

Static config produces correct 34-key split with mirrored halves and
thumbs. layoutToErgogen still has alignment bugs (column shifts off,
thumbs floating) — left for the next iteration. The infrastructure for
fast iteration is in place: edit math → save → click build → see render.

devenv.nix updated: dev (server), ergogen (one-shot), render (CLI render).
Parts:
- added D10: , ceoloide:diode_tht_sod123, B.Cu at (140.5, -34.9)
- added D11: , ceoloide:diode_tht_sod123, B.Cu at (150.1, -12.7)
- added D12: , ceoloide:diode_tht_sod123, B.Cu at (159.6, 9.44)
- added D13: , ceoloide:diode_tht_sod123, B.Cu at (159.5, -32.9)
- added D14: , ceoloide:diode_tht_sod123, B.Cu at (169.1, -8.89)
- added D15: , ceoloide:diode_tht_sod123, B.Cu at (178.6, 15.2)
- added D16: , ceoloide:diode_tht_sod123, B.Cu at (162.1, -11.2)
- added D17: , ceoloide:diode_tht_sod123, B.Cu at (201.2, -14.0)
- added D18: , ceoloide:diode_tht_sod123, B.Cu at (428.5, -23.8)
- added D19: , ceoloide:diode_tht_sod123, B.Cu at (419.0, 9.39)
- added D2: , ceoloide:diode_tht_sod123, B.Cu at (93.1, 9.39)
- added D20: , ceoloide:diode_tht_sod123, B.Cu at (409.4, 42.6)
- added D21: , ceoloide:diode_tht_sod123, B.Cu at (409.5, -34.9)
- added D22: , ceoloide:diode_tht_sod123, B.Cu at (400.0, -12.7)
- added D23: , ceoloide:diode_tht_sod123, B.Cu at (390.4, 9.44)
- added D24: , ceoloide:diode_tht_sod123, B.Cu at (390.5, -37.9)
- added D25: , ceoloide:diode_tht_sod123, B.Cu at (381.0, -18.8)
- added D26: , ceoloide:diode_tht_sod123, B.Cu at (371.4, 0.30)
- added D27: , ceoloide:diode_tht_sod123, B.Cu at (371.5, -34.9)
- added D28: , ceoloide:diode_tht_sod123, B.Cu at (362.0, -12.7)
- added D29: , ceoloide:diode_tht_sod123, B.Cu at (352.4, 9.44)
- added D3: , ceoloide:diode_tht_sod123, B.Cu at (102.6, 42.6)
- added D30: , ceoloide:diode_tht_sod123, B.Cu at (352.5, -32.9)
- added D31: , ceoloide:diode_tht_sod123, B.Cu at (343.0, -8.89)
- added D32: , ceoloide:diode_tht_sod123, B.Cu at (333.4, 15.2)
- added D33: , ceoloide:diode_tht_sod123, B.Cu at (349.9, -11.2)
- added D34: , ceoloide:diode_tht_sod123, B.Cu at (310.9, -14.0)
- added D4: , ceoloide:diode_tht_sod123, B.Cu at (102.5, -34.9)
- added D5: , ceoloide:diode_tht_sod123, B.Cu at (112.1, -12.7)
- added D6: , ceoloide:diode_tht_sod123, B.Cu at (121.6, 9.44)
- added D7: , ceoloide:diode_tht_sod123, B.Cu at (121.5, -37.9)
- added D8: , ceoloide:diode_tht_sod123, B.Cu at (131.1, -18.8)
- added D9: , ceoloide:diode_tht_sod123, B.Cu at (140.6, 0.30)
- added LED10: , ceoloide:led_SK6812mini-e (per-keysingle-side), B.Cu at (146.5, -43.8)
- added LED11: , ceoloide:led_SK6812mini-e (per-keysingle-side), B.Cu at (156.1, -21.6)
- added LED12: , ceoloide:led_SK6812mini-e (per-keysingle-side), B.Cu at (165.6, 0.51)
- added LED13: , ceoloide:led_SK6812mini-e (per-keysingle-side), B.Cu at (165.5, -41.9)
- added LED14: , ceoloide:led_SK6812mini-e (per-keysingle-side), B.Cu at (175.1, -17.8)
- added LED15: , ceoloide:led_SK6812mini-e (per-keysingle-side), B.Cu at (184.6, 6.23)
- added LED16: , ceoloide:led_SK6812mini-e (per-keysingle-side), B.Cu at (165.7, -21.3)
- added LED17: , ceoloide:led_SK6812mini-e (per-keysingle-side), B.Cu at (203.6, -24.5)
- added LED18: , ceoloide:led_SK6812mini-e (per-keysingle-side), B.Cu at (422.5, -32.7)
- added LED19: , ceoloide:led_SK6812mini-e (per-keysingle-side), B.Cu at (413.0, 0.46)
- added LED2: , ceoloide:led_SK6812mini-e (per-keysingle-side), B.Cu at (99.1, 0.46)
- added LED20: , ceoloide:led_SK6812mini-e (per-keysingle-side), B.Cu at (403.4, 33.7)
- added LED21: , ceoloide:led_SK6812mini-e (per-keysingle-side), B.Cu at (403.5, -43.8)
- added LED22: , ceoloide:led_SK6812mini-e (per-keysingle-side), B.Cu at (394.0, -21.6)
- added LED23: , ceoloide:led_SK6812mini-e (per-keysingle-side), B.Cu at (384.4, 0.51)
- added LED24: , ceoloide:led_SK6812mini-e (per-keysingle-side), B.Cu at (384.5, -46.8)
- added LED25: , ceoloide:led_SK6812mini-e (per-keysingle-side), B.Cu at (375.0, -27.7)
- added LED26: , ceoloide:led_SK6812mini-e (per-keysingle-side), B.Cu at (365.4, -8.63)
- added LED27: , ceoloide:led_SK6812mini-e (per-keysingle-side), B.Cu at (365.5, -43.8)
- added LED28: , ceoloide:led_SK6812mini-e (per-keysingle-side), B.Cu at (356.0, -21.6)
- added LED29: , ceoloide:led_SK6812mini-e (per-keysingle-side), B.Cu at (346.4, 0.51)
- added LED3: , ceoloide:led_SK6812mini-e (per-keysingle-side), B.Cu at (108.6, 33.7)
- added LED30: , ceoloide:led_SK6812mini-e (per-keysingle-side), B.Cu at (346.5, -41.9)
- added LED31: , ceoloide:led_SK6812mini-e (per-keysingle-side), B.Cu at (337.0, -17.8)
- added LED32: , ceoloide:led_SK6812mini-e (per-keysingle-side), B.Cu at (327.4, 6.23)
- added LED33: , ceoloide:led_SK6812mini-e (per-keysingle-side), B.Cu at (346.3, -21.3)
- added LED34: , ceoloide:led_SK6812mini-e (per-keysingle-side), B.Cu at (308.5, -24.5)
- added LED4: , ceoloide:led_SK6812mini-e (per-keysingle-side), B.Cu at (108.5, -43.8)
- added LED5: , ceoloide:led_SK6812mini-e (per-keysingle-side), B.Cu at (118.1, -21.6)
- added LED6: , ceoloide:led_SK6812mini-e (per-keysingle-side), B.Cu at (127.6, 0.51)
- added LED7: , ceoloide:led_SK6812mini-e (per-keysingle-side), B.Cu at (127.5, -46.8)
- added LED8: , ceoloide:led_SK6812mini-e (per-keysingle-side), B.Cu at (137.1, -27.7)
- added LED9: , ceoloide:led_SK6812mini-e (per-keysingle-side), B.Cu at (146.6, -8.63)
- added S10: , ceoloide:switch_choc_v1_v2, F.Cu at (146.5, -38.9)
- added S11: , ceoloide:switch_choc_v1_v2, F.Cu at (156.1, -16.7)
- added S12: , ceoloide:switch_choc_v1_v2, F.Cu at (165.6, 5.44)
- added S13: , ceoloide:switch_choc_v1_v2, F.Cu at (165.5, -36.9)
- added S14: , ceoloide:switch_choc_v1_v2, F.Cu at (175.1, -12.9)
- added S15: , ceoloide:switch_choc_v1_v2, F.Cu at (184.6, 11.2)
- added S16: , ceoloide:switch_choc_v1_v2, F.Cu at (166.9, -16.5)
- added S17: , ceoloide:switch_choc_v1_v2, F.Cu at (205.3, -19.9)
- added S18: , ceoloide:switch_choc_v1_v2, F.Cu at (422.5, -27.8)
- added S19: , ceoloide:switch_choc_v1_v2, F.Cu at (413.0, 5.39)
- added S2: , ceoloide:switch_choc_v1_v2, F.Cu at (99.1, 5.39)
- added S20: , ceoloide:switch_choc_v1_v2, F.Cu at (403.4, 38.6)
- added S21: , ceoloide:switch_choc_v1_v2, F.Cu at (403.5, -38.9)
- added S22: , ceoloide:switch_choc_v1_v2, F.Cu at (394.0, -16.7)
- added S23: , ceoloide:switch_choc_v1_v2, F.Cu at (384.4, 5.44)
- added S24: , ceoloide:switch_choc_v1_v2, F.Cu at (384.5, -41.9)
- added S25: , ceoloide:switch_choc_v1_v2, F.Cu at (375.0, -22.8)
- added S26: , ceoloide:switch_choc_v1_v2, F.Cu at (365.4, -3.70)
- added S27: , ceoloide:switch_choc_v1_v2, F.Cu at (365.5, -38.9)
- added S28: , ceoloide:switch_choc_v1_v2, F.Cu at (356.0, -16.7)
- added S29: , ceoloide:switch_choc_v1_v2, F.Cu at (346.4, 5.44)
- added S3: , ceoloide:switch_choc_v1_v2, F.Cu at (108.6, 38.6)
- added S30: , ceoloide:switch_choc_v1_v2, F.Cu at (346.5, -36.9)
- added S31: , ceoloide:switch_choc_v1_v2, F.Cu at (337.0, -12.9)
- added S32: , ceoloide:switch_choc_v1_v2, F.Cu at (327.4, 11.2)
- added S33: , ceoloide:switch_choc_v1_v2, F.Cu at (345.1, -16.5)
- added S34: , ceoloide:switch_choc_v1_v2, F.Cu at (306.7, -19.9)
- added S4: , ceoloide:switch_choc_v1_v2, F.Cu at (108.5, -38.9)
- added S5: , ceoloide:switch_choc_v1_v2, F.Cu at (118.1, -16.7)
- added S6: , ceoloide:switch_choc_v1_v2, F.Cu at (127.6, 5.44)
- added S7: , ceoloide:switch_choc_v1_v2, F.Cu at (127.5, -41.9)
- added S8: , ceoloide:switch_choc_v1_v2, F.Cu at (137.1, -22.8)
- added S9: , ceoloide:switch_choc_v1_v2, F.Cu at (146.6, -3.70)
- moved D1 45.3 mm to (83.5, -23.8)
- moved LED1 45.3 mm to (89.5, -32.7)
- moved S1 45.3 mm to (89.5, -27.8)
Connections:
- net DIN renamed led_din_matrix_c0_r0
- net DOUT renamed led_dout_matrix_c0_r0
- D1 pad 1: NET_X -> ROW0
- D1 pad 2: COL -> c0_r0
- S1 pad 1: COL -> COL0
- S1 pad 2: ROW -> c0_r0
Other:
- board size 22 x 22 mm -> 357 x 104.5 mm

Commit message: feat(pcb): atlas PCB from ergogen webtool pipeline; tools/ goes private
Drops the staged ergogen + webtool tooling out of the public branch
(tools/ is gitignored from here on) and commits only the generated
KiCad PCB plus supporting BOM/docs. The .kicad_pcb is the totem-choc
output of the cap-configurator pipeline — keys-only board, mirrored
halves, trackpoint cutout between the top-right key cluster, no MCU
(placed by hand in KiCad).

- .gitignore: tools/ + devenv state private; keep KiCad/output cruft
  out of git (kicad_prl, autosaves, generated step/dxf/stl, gerbers,
  Fab-Toolkit zips, IDE/OS noise)
- pcb/keyboard.svg, keyboard-outline.svg, keyboard-plate.svg removed
  (pre-pipeline relics — outline now comes from ergogen)
- package.json moved to tools/ so root no longer advertises a node
  project
- pcb/kicad/keyboard.kicad_pcb refreshed from the latest ergogen run
Parts:
- added D35: , ceoloide:diode_tht_sod123, B.Cu at (234.7, -64.1)
- added D36: , ceoloide:diode_tht_sod123, B.Cu at (257.7, -12.1)
- added D37: , ceoloide:diode_tht_sod123, B.Cu at (236.9, -7.93)
- added D38: , ceoloide:diode_tht_sod123, B.Cu at (218.0, 1.19)
- added LED35: , ceoloide:led_SK6812mini-e (per-keysingle-side), B.Cu at (240.7, -65.0)
- added LED36: , ceoloide:led_SK6812mini-e (per-keysingle-side), B.Cu at (263.7, -13.0)
- added LED37: , ceoloide:led_SK6812mini-e (per-keysingle-side), B.Cu at (242.5, -10.4)
- added LED38: , ceoloide:led_SK6812mini-e (per-keysingle-side), B.Cu at (222.7, -2.61)
- added MH1: , ceoloide:mounting_hole_npth, F.Cu at (161.0, -52.9)
- added MH2: , ceoloide:mounting_hole_npth, F.Cu at (249.7, -52.9)
- added MH3: , ceoloide:mounting_hole_npth, F.Cu at (161.0, -62.4)
- added MH4: , ceoloide:mounting_hole_npth, F.Cu at (249.7, -62.4)
- added MH5: , ceoloide:mounting_hole_npth, F.Cu at (161.0, -43.4)
- added MH6: , ceoloide:mounting_hole_npth, F.Cu at (249.7, -43.4)
- added S35: , ceoloide:switch_choc_v1_v2, B.Cu at (185.6, 1.66)
- added S36: , ceoloide:switch_choc_v1_v2, B.Cu at (263.7, -8.11)
- added S37: , ceoloide:switch_choc_v1_v2, B.Cu at (243.8, -5.62)
- added S38: , ceoloide:switch_choc_v1_v2, B.Cu at (225.2, 1.66)
- S1, S10, S11, S12, S13, S14, S15, S16, S17, S18, S19, S2, S20, S21, S22, S23, S24, S25, S26, S27, S28, S29, S3, S30, S31, S32, S33, S34, S4, S5, S6, S7, S8, S9: moved to B.Cu
- moved D18 266.6 mm to (162.2, -11.0), turned to 75 degrees
- moved LED18 255.2 mm to (168.2, -10.4), turned to -15 degrees
- moved D19 237.0 mm to (182.4, -4.81), turned to 60 degrees
- moved LED19 225.0 mm to (188.0, -2.61), turned to -30 degrees
- moved S33 198.3 mm to (147.0, -8.11), turned to 180 degrees
- moved S34 140.4 mm to (167.0, -5.62), turned to 165 degrees
- moved S17 125.4 mm to (330.7, -16.4), turned to -190 degrees
- moved S20 120.2 mm to (317.6, -45.5), turned to -190 degrees
- moved D29 117.7 mm to (270.7, -75.2), turned to 90 degrees
- moved D33 116.8 mm to (234.7, -30.1), turned to 90 degrees
- moved D32 115.0 mm to (252.7, -66.7), turned to 90 degrees
- moved S32 112.2 mm to (240.7, -60.1), turned to -180 degrees
- moved S18 112.0 mm to (311.7, -12.0), turned to -190 degrees
- moved S26 111.5 mm to (276.7, -71.2), turned to -180 degrees
- moved S29 111.1 mm to (258.7, -62.7), turned to -180 degrees
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Connections:
- net led_din_mirror_matrix_c0_r1 renamed led_dout_thumbs_t2_thumb
- net led_din_mirror_thumbs_t0_thumb renamed led_dout_mirror_matrix_c5_r0
- net led_din_mirror_thumbs_t1_thumb renamed led_dout_mirror_matrix_c5_r1
- net led_dout_mirror_matrix_c0_r1 renamed led_din_thumbs_t2_thumb
- net led_dout_mirror_thumbs_t0_thumb renamed led_din_mirror_matrix_c5_r0
- net led_dout_mirror_thumbs_t1_thumb renamed led_din_mirror_matrix_c5_r1
- D10 pad 1: ROW0 -> ROW2
- D10 pad 2: c3_r0 -> c3_r2
- D11 pad 1: ROW1 -> ROW0
- D11 pad 2: c3_r1 -> c4_r0
- D12 pad 1: ROW2 -> ROW1
- D12 pad 2: c3_r2 -> c4_r1
- D13 pad 1: ROW0 -> ROW2
- D13 pad 2: c4_r0 -> c4_r2
- D14 pad 1: ROW1 -> ROW0
- D14 pad 2: c4_r1 -> c5_r0
- D15 pad 1: ROW2 -> ROW1
- D15 pad 2: c4_r2 -> c5_r1
- D16 pad 1: TROW0 -> ROW2
- D16 pad 2: t0_thumb -> c5_r2
- D17 pad 2: t1_thumb -> t0_thumb
- D18 pad 1: ROW0 -> TROW0
- D18 pad 2: mirror_c0_r0 -> t1_thumb
- D19 pad 1: ROW1 -> TROW0
- D19 pad 2: mirror_c0_r1 -> t2_thumb
- D2 pad 1: ROW1 -> ROW0
- D2 pad 2: c0_r1 -> c1_r0
- D20 pad 1: ROW2 -> ROW0
- D20 pad 2: mirror_c0_r2 -> mirror_c0_r0
- D3 pad 1: ROW2 -> ROW1
- D3 pad 2: c0_r2 -> c1_r1
- D33 pad 1: TROW0 -> ROW0
- D33 pad 2: mirror_t0_thumb -> mirror_c5_r0
- D34 pad 1: TROW0 -> ROW1
- D34 pad 2: mirror_t1_thumb -> mirror_c5_r1
- D4 pad 1: ROW0 -> ROW2
- D4 pad 2: c1_r0 -> c1_r2
- D5 pad 1: ROW1 -> ROW0
- D5 pad 2: c1_r1 -> c2_r0
- D6 pad 1: ROW2 -> ROW1
- D6 pad 2: c1_r2 -> c2_r1
- D7 pad 1: ROW0 -> ROW2
- D7 pad 2: c2_r0 -> c2_r2
- D8 pad 1: ROW1 -> ROW0
- D8 pad 2: c2_r1 -> c3_r0
- D9 pad 1: ROW2 -> ROW1
- D9 pad 2: c2_r2 -> c3_r1
- LED1 pad 2: led_dout_matrix_c0_r0 -> led_din_matrix_c0_r0
- LED1 pad 4: led_din_matrix_c0_r0 -> led_dout_matrix_c0_r0
- LED10 pad 2: led_dout_matrix_c3_r0 -> led_din_matrix_c3_r2
- LED10 pad 4: led_din_matrix_c3_r0 -> led_dout_matrix_c3_r2
- LED11 pad 2: led_dout_matrix_c3_r1 -> led_din_matrix_c4_r0
- LED11 pad 4: led_din_matrix_c3_r1 -> led_dout_matrix_c4_r0
- LED12 pad 2: led_dout_matrix_c3_r2 -> led_din_matrix_c4_r1
- LED12 pad 4: led_din_matrix_c3_r2 -> led_dout_matrix_c4_r1
- LED13 pad 2: led_dout_matrix_c4_r0 -> led_din_matrix_c4_r2
- LED13 pad 4: led_din_matrix_c4_r0 -> led_dout_matrix_c4_r2
- LED14 pad 2: led_dout_matrix_c4_r1 -> led_din_matrix_c5_r0
- LED14 pad 4: led_din_matrix_c4_r1 -> led_dout_matrix_c5_r0
- LED15 pad 2: led_dout_matrix_c4_r2 -> led_din_matrix_c5_r1
- LED15 pad 4: led_din_matrix_c4_r2 -> led_dout_matrix_c5_r1
- LED16 pad 2: led_dout_thumbs_t0_thumb -> led_din_matrix_c5_r2
- LED16 pad 4: led_din_thumbs_t0_thumb -> led_dout_matrix_c5_r2
- LED17 pad 2: led_dout_thumbs_t1_thumb -> led_din_thumbs_t0_thumb
- LED17 pad 4: led_din_thumbs_t1_thumb -> led_dout_thumbs_t0_thumb
- LED18 pad 2: led_dout_mirror_matrix_c0_r0 -> led_din_thumbs_t1_thumb
- LED18 pad 4: led_din_mirror_matrix_c0_r0 -> led_dout_thumbs_t1_thumb
- LED2 pad 2: led_dout_matrix_c0_r1 -> led_din_matrix_c1_r0
- LED2 pad 4: led_din_matrix_c0_r1 -> led_dout_matrix_c1_r0
- LED20 pad 2: led_dout_mirror_matrix_c0_r2 -> led_din_mirror_matrix_c0_r0
- LED20 pad 4: led_din_mirror_matrix_c0_r2 -> led_dout_mirror_matrix_c0_r0
- LED21 pad 2: led_dout_mirror_matrix_c1_r0 -> led_din_mirror_matrix_c1_r0
- LED21 pad 4: led_din_mirror_matrix_c1_r0 -> led_dout_mirror_matrix_c1_r0
- LED22 pad 2: led_dout_mirror_matrix_c1_r1 -> led_din_mirror_matrix_c1_r1
- LED22 pad 4: led_din_mirror_matrix_c1_r1 -> led_dout_mirror_matrix_c1_r1
- LED23 pad 2: led_dout_mirror_matrix_c1_r2 -> led_din_mirror_matrix_c1_r2
- LED23 pad 4: led_din_mirror_matrix_c1_r2 -> led_dout_mirror_matrix_c1_r2
- LED24 pad 2: led_dout_mirror_matrix_c2_r0 -> led_din_mirror_matrix_c2_r0
- LED24 pad 4: led_din_mirror_matrix_c2_r0 -> led_dout_mirror_matrix_c2_r0
- LED25 pad 2: led_dout_mirror_matrix_c2_r1 -> led_din_mirror_matrix_c2_r1
- LED25 pad 4: led_din_mirror_matrix_c2_r1 -> led_dout_mirror_matrix_c2_r1
- LED26 pad 2: led_dout_mirror_matrix_c2_r2 -> led_din_mirror_matrix_c2_r2
- LED26 pad 4: led_din_mirror_matrix_c2_r2 -> led_dout_mirror_matrix_c2_r2
- LED27 pad 2: led_dout_mirror_matrix_c3_r0 -> led_din_mirror_matrix_c3_r0
- LED27 pad 4: led_din_mirror_matrix_c3_r0 -> led_dout_mirror_matrix_c3_r0
- LED28 pad 2: led_dout_mirror_matrix_c3_r1 -> led_din_mirror_matrix_c3_r1
- LED28 pad 4: led_din_mirror_matrix_c3_r1 -> led_dout_mirror_matrix_c3_r1
- LED29 pad 2: led_dout_mirror_matrix_c3_r2 -> led_din_mirror_matrix_c3_r2
- LED29 pad 4: led_din_mirror_matrix_c3_r2 -> led_dout_mirror_matrix_c3_r2
- LED3 pad 2: led_dout_matrix_c0_r2 -> led_din_matrix_c1_r1
- LED3 pad 4: led_din_matrix_c0_r2 -> led_dout_matrix_c1_r1
- LED30 pad 2: led_dout_mirror_matrix_c4_r0 -> led_din_mirror_matrix_c4_r0
- LED30 pad 4: led_din_mirror_matrix_c4_r0 -> led_dout_mirror_matrix_c4_r0
- LED31 pad 2: led_dout_mirror_matrix_c4_r1 -> led_din_mirror_matrix_c4_r1
- LED31 pad 4: led_din_mirror_matrix_c4_r1 -> led_dout_mirror_matrix_c4_r1
- LED32 pad 2: led_dout_mirror_matrix_c4_r2 -> led_din_mirror_matrix_c4_r2
- LED32 pad 4: led_din_mirror_matrix_c4_r2 -> led_dout_mirror_matrix_c4_r2
- LED4 pad 2: led_dout_matrix_c1_r0 -> led_din_matrix_c1_r2
- LED4 pad 4: led_din_matrix_c1_r0 -> led_dout_matrix_c1_r2
- LED5 pad 2: led_dout_matrix_c1_r1 -> led_din_matrix_c2_r0
- LED5 pad 4: led_din_matrix_c1_r1 -> led_dout_matrix_c2_r0
- LED6 pad 2: led_dout_matrix_c1_r2 -> led_din_matrix_c2_r1
- LED6 pad 4: led_din_matrix_c1_r2 -> led_dout_matrix_c2_r1
- LED7 pad 2: led_dout_matrix_c2_r0 -> led_din_matrix_c2_r2
- LED7 pad 4: led_din_matrix_c2_r0 -> led_dout_matrix_c2_r2
- LED8 pad 2: led_dout_matrix_c2_r1 -> led_din_matrix_c3_r0
- LED8 pad 4: led_din_matrix_c2_r1 -> led_dout_matrix_c3_r0
- LED9 pad 2: led_dout_matrix_c2_r2 -> led_din_matrix_c3_r1
- LED9 pad 4: led_din_matrix_c2_r2 -> led_dout_matrix_c3_r1
- S10 pad 2: c3_r0 -> c3_r2
- S11 pad 1: COL3 -> COL4
- S11 pad 2: c3_r1 -> c4_r0
- S12 pad 1: COL3 -> COL4
- S12 pad 2: c3_r2 -> c4_r1
- S13 pad 2: c4_r0 -> c4_r2
- S14 pad 1: COL4 -> COL5
- S14 pad 2: c4_r1 -> c5_r0
- S15 pad 1: COL4 -> COL5
- S15 pad 2: c4_r2 -> c5_r1
- S16 pad 1: TCOL0 -> COL5
- S16 pad 2: t0_thumb -> c5_r2
- S17 pad 1: TCOL1 -> COL0
- S17 pad 2: t1_thumb -> mirror_c0_r0
- S18 pad 1: COL0 -> COL1
- S18 pad 2: mirror_c0_r0 -> mirror_c1_r0
- S19 pad 1: COL0 -> COL1
- S19 pad 2: mirror_c0_r1 -> mirror_c1_r1
- S2 pad 1: COL0 -> COL1
- S2 pad 2: c0_r1 -> c1_r0
- S20 pad 1: COL0 -> COL1
- S20 pad 2: mirror_c0_r2 -> mirror_c1_r2
- S21 pad 1: COL1 -> COL2
- S21 pad 2: mirror_c1_r0 -> mirror_c2_r0
- S22 pad 1: COL1 -> COL2
- S22 pad 2: mirror_c1_r1 -> mirror_c2_r1
- S23 pad 1: COL1 -> COL2
- S23 pad 2: mirror_c1_r2 -> mirror_c2_r2
- S24 pad 1: COL2 -> COL3
- S24 pad 2: mirror_c2_r0 -> mirror_c3_r0
- S25 pad 1: COL2 -> COL3
- S25 pad 2: mirror_c2_r1 -> mirror_c3_r1
- S26 pad 1: COL2 -> COL3
- S26 pad 2: mirror_c2_r2 -> mirror_c3_r2
- S27 pad 1: COL3 -> COL4
- S27 pad 2: mirror_c3_r0 -> mirror_c4_r0
- S28 pad 1: COL3 -> COL4
- S28 pad 2: mirror_c3_r1 -> mirror_c4_r1
- S29 pad 1: COL3 -> COL4
- S29 pad 2: mirror_c3_r2 -> mirror_c4_r2
- S3 pad 1: COL0 -> COL1
- S3 pad 2: c0_r2 -> c1_r1
- S30 pad 1: COL4 -> COL5
- S30 pad 2: mirror_c4_r0 -> mirror_c5_r0
- S31 pad 1: COL4 -> COL5
- S31 pad 2: mirror_c4_r1 -> mirror_c5_r1
- S32 pad 1: COL4 -> COL5
- S32 pad 2: mirror_c4_r2 -> mirror_c5_r2
- S33 pad 2: mirror_t0_thumb -> t0_thumb
- S34 pad 2: mirror_t1_thumb -> t1_thumb
- S4 pad 2: c1_r0 -> c1_r2
- S5 pad 1: COL1 -> COL2
- S5 pad 2: c1_r1 -> c2_r0
- S6 pad 1: COL1 -> COL2
- S6 pad 2: c1_r2 -> c2_r1
- S7 pad 2: c2_r0 -> c2_r2
- S8 pad 1: COL2 -> COL3
- S8 pad 2: c2_r1 -> c3_r0
- S9 pad 1: COL2 -> COL3
- S9 pad 2: c2_r2 -> c3_r1
Other:
- board size 357 x 104.5 mm -> 275.6 x 98.2 mm

Commit message: pcb: regenerate keyboard.kicad_pcb from ergogen pipeline
Net topology collapsed/renumbered by the latest pipeline run; no
schematic changes intended.
Parts:
- removed D35, D36, D37, D38: , ceoloide:diode_tht_sod123
- removed LED35, LED36, LED37, LED38: , ceoloide:led_SK6812mini-e (per-keysingle-side)
- removed S35, S36, S37, S38: , ceoloide:switch_choc_v1_v2
- moved S19 228.1 mm to (89.5, -65.9), turned to 180 degrees
- moved S20 211.3 mm to (108.6, -77.0), turned to 180 degrees
- moved S6 203.1 mm to (317.0, -27.8), turned to -180 degrees
- moved S7 185.9 mm to (298.0, -38.9), turned to -180 degrees
- moved S21 175.5 mm to (127.6, -80.0), turned to 180 degrees
- moved S22 153.0 mm to (146.7, -77.0), turned to 180 degrees
- moved LED18 150.5 mm to (317.0, -32.7), turned to 0 degrees
- moved D18 150.3 mm to (311.0, -31.8), turned to 90 degrees
- moved S15 147.1 mm to (317.0, -46.9)
- moved S8 145.0 mm to (278.9, -41.9)
- moved LED19 138.0 mm to (317.0, -51.8), turned to 0 degrees
- moved D19 136.6 mm to (311.0, -50.9), turned to 90 degrees
- moved S23 132.3 mm to (165.7, -75.0), turned to 180 degrees
- moved S16 128.0 mm to (298.0, -57.9)
- moved S9 126.8 mm to (259.9, -38.9)
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Connections:
- net led_din_thumbs_t2_thumb renamed led_din_mirror_matrix_c0_r1
- net led_dout_thumbs_t2_thumb renamed led_dout_mirror_matrix_c0_r1
- D10 pad 1: ROW2 -> ROW0
- D10 pad 2: c3_r2 -> c3_r0
- D11 pad 1: ROW0 -> ROW1
- D11 pad 2: c4_r0 -> c3_r1
- D12 pad 1: ROW1 -> ROW2
- D12 pad 2: c4_r1 -> c3_r2
- D13 pad 1: ROW2 -> ROW0
- D13 pad 2: c4_r2 -> c4_r0
- D14 pad 1: ROW0 -> ROW1
- D14 pad 2: c5_r0 -> c4_r1
- D15 pad 1: ROW1 -> ROW2
- D15 pad 2: c5_r1 -> c4_r2
- D16 pad 1: ROW2 -> TROW0
- D16 pad 2: c5_r2 -> t0_thumb
- D17 pad 2: t0_thumb -> t1_thumb
- D18 pad 1: TROW0 -> ROW0
- D18 pad 2: t1_thumb -> mirror_c0_r0
- D19 pad 1: TROW0 -> ROW1
- D19 pad 2: t2_thumb -> mirror_c0_r1
- D2 pad 1: ROW0 -> ROW1
- D2 pad 2: c1_r0 -> c0_r1
- D20 pad 1: ROW0 -> ROW2
- D20 pad 2: mirror_c0_r0 -> mirror_c0_r2
- D3 pad 1: ROW1 -> ROW2
- D3 pad 2: c1_r1 -> c0_r2
- D33 pad 1: ROW0 -> TROW0
- D33 pad 2: mirror_c5_r0 -> mirror_t0_thumb
- D34 pad 1: ROW1 -> TROW0
- D34 pad 2: mirror_c5_r1 -> mirror_t1_thumb
- D4 pad 1: ROW2 -> ROW0
- D4 pad 2: c1_r2 -> c1_r0
- D5 pad 1: ROW0 -> ROW1
- D5 pad 2: c2_r0 -> c1_r1
- D6 pad 1: ROW1 -> ROW2
- D6 pad 2: c2_r1 -> c1_r2
- D7 pad 1: ROW2 -> ROW0
- D7 pad 2: c2_r2 -> c2_r0
- D8 pad 1: ROW0 -> ROW1
- D8 pad 2: c3_r0 -> c2_r1
- D9 pad 1: ROW1 -> ROW2
- D9 pad 2: c3_r1 -> c2_r2
- LED10 pad 2: led_din_matrix_c3_r2 -> led_din_matrix_c3_r0
- LED10 pad 4: led_dout_matrix_c3_r2 -> led_dout_matrix_c3_r0
- LED11 pad 2: led_din_matrix_c4_r0 -> led_din_matrix_c3_r1
- LED11 pad 4: led_dout_matrix_c4_r0 -> led_dout_matrix_c3_r1
- LED12 pad 2: led_din_matrix_c4_r1 -> led_din_matrix_c3_r2
- LED12 pad 4: led_dout_matrix_c4_r1 -> led_dout_matrix_c3_r2
- LED13 pad 2: led_din_matrix_c4_r2 -> led_din_matrix_c4_r0
- LED13 pad 4: led_dout_matrix_c4_r2 -> led_dout_matrix_c4_r0
- LED14 pad 2: led_din_matrix_c5_r0 -> led_din_matrix_c4_r1
- LED14 pad 4: led_dout_matrix_c5_r0 -> led_dout_matrix_c4_r1
- LED15 pad 2: led_din_matrix_c5_r1 -> led_din_matrix_c4_r2
- LED15 pad 4: led_dout_matrix_c5_r1 -> led_dout_matrix_c4_r2
- LED16 pad 2: led_din_matrix_c5_r2 -> led_din_thumbs_t0_thumb
- LED16 pad 4: led_dout_matrix_c5_r2 -> led_dout_thumbs_t0_thumb
- LED17 pad 2: led_din_thumbs_t0_thumb -> led_din_thumbs_t1_thumb
- LED17 pad 4: led_dout_thumbs_t0_thumb -> led_dout_thumbs_t1_thumb
- LED18 pad 2: led_din_thumbs_t1_thumb -> led_din_mirror_matrix_c0_r0
- LED18 pad 4: led_dout_thumbs_t1_thumb -> led_dout_mirror_matrix_c0_r0
- LED2 pad 2: led_din_matrix_c1_r0 -> led_din_matrix_c0_r1
- LED2 pad 4: led_dout_matrix_c1_r0 -> led_dout_matrix_c0_r1
- LED20 pad 2: led_din_mirror_matrix_c0_r0 -> led_din_mirror_matrix_c0_r2
- LED20 pad 4: led_dout_mirror_matrix_c0_r0 -> led_dout_mirror_matrix_c0_r2
- LED3 pad 2: led_din_matrix_c1_r1 -> led_din_matrix_c0_r2
- LED3 pad 4: led_dout_matrix_c1_r1 -> led_dout_matrix_c0_r2
- LED33 pad 2: led_din_mirror_matrix_c5_r0 -> led_din_mirror_thumbs_t0_thumb
- LED33 pad 4: led_dout_mirror_matrix_c5_r0 -> led_dout_mirror_thumbs_t0_thumb
- LED34 pad 2: led_din_mirror_matrix_c5_r1 -> led_din_mirror_thumbs_t1_thumb
- LED34 pad 4: led_dout_mirror_matrix_c5_r1 -> led_dout_mirror_thumbs_t1_thumb
- LED4 pad 2: led_din_matrix_c1_r2 -> led_din_matrix_c1_r0
- LED4 pad 4: led_dout_matrix_c1_r2 -> led_dout_matrix_c1_r0
- LED5 pad 2: led_din_matrix_c2_r0 -> led_din_matrix_c1_r1
- LED5 pad 4: led_dout_matrix_c2_r0 -> led_dout_matrix_c1_r1
- LED6 pad 2: led_din_matrix_c2_r1 -> led_din_matrix_c1_r2
- LED6 pad 4: led_dout_matrix_c2_r1 -> led_dout_matrix_c1_r2
- LED7 pad 2: led_din_matrix_c2_r2 -> led_din_matrix_c2_r0
- LED7 pad 4: led_dout_matrix_c2_r2 -> led_dout_matrix_c2_r0
- LED8 pad 2: led_din_matrix_c3_r0 -> led_din_matrix_c2_r1
- LED8 pad 4: led_dout_matrix_c3_r0 -> led_dout_matrix_c2_r1
- LED9 pad 2: led_din_matrix_c3_r1 -> led_din_matrix_c2_r2
- LED9 pad 4: led_dout_matrix_c3_r1 -> led_dout_matrix_c2_r2
- S10 pad 1: COL3 -> COL4
- S10 pad 2: c3_r2 -> mirror_c4_r0
- S11 pad 1: COL4 -> COL0
- S11 pad 2: c4_r0 -> c0_r1
- S12 pad 1: COL4 -> COL1
- S12 pad 2: c4_r1 -> c1_r1
- S13 pad 1: COL4 -> COL2
- S13 pad 2: c4_r2 -> c2_r1
- S14 pad 1: COL5 -> COL4
- S14 pad 2: c5_r0 -> c4_r1
- S15 pad 1: COL5 -> COL0
- S15 pad 2: c5_r1 -> mirror_c0_r1
- S16 pad 1: COL5 -> COL1
- S16 pad 2: c5_r2 -> mirror_c1_r1
- S17 pad 1: COL0 -> COL2
- S17 pad 2: mirror_c0_r0 -> mirror_c2_r1
- S18 pad 1: COL1 -> COL4
- S18 pad 2: mirror_c1_r0 -> mirror_c4_r1
- S19 pad 1: COL1 -> COL0
- S19 pad 2: mirror_c1_r1 -> c0_r2
- S20 pad 2: mirror_c1_r2 -> c1_r2
- S21 pad 2: mirror_c2_r0 -> c2_r2
- S22 pad 1: COL2 -> COL3
- S22 pad 2: mirror_c2_r1 -> c3_r2
- S23 pad 1: COL2 -> COL4
- S23 pad 2: mirror_c2_r2 -> c4_r2
- S24 pad 1: COL3 -> COL0
- S24 pad 2: mirror_c3_r0 -> mirror_c0_r2
- S25 pad 1: COL3 -> COL1
- S25 pad 2: mirror_c3_r1 -> mirror_c1_r2
- S26 pad 1: COL3 -> COL2
- S26 pad 2: mirror_c3_r2 -> mirror_c2_r2
- S27 pad 1: COL4 -> COL3
- S27 pad 2: mirror_c4_r0 -> mirror_c3_r2
- S28 pad 2: mirror_c4_r1 -> mirror_c4_r2
- S29 pad 1: COL4 -> COL3
- S29 pad 2: mirror_c4_r2 -> c3_r1
- S3 pad 1: COL1 -> COL2
- S3 pad 2: c1_r1 -> c2_r0
- S30 pad 1: COL5 -> COL3
- S30 pad 2: mirror_c5_r0 -> mirror_c3_r1
- S31 pad 1: COL5 -> TCOL0
- S31 pad 2: mirror_c5_r1 -> t0_thumb
- S32 pad 1: COL5 -> TCOL1
- S32 pad 2: mirror_c5_r2 -> t1_thumb
- S33 pad 2: t0_thumb -> mirror_t0_thumb
- S34 pad 2: t1_thumb -> mirror_t1_thumb
- S4 pad 1: COL1 -> COL3
- S4 pad 2: c1_r2 -> c3_r0
- S5 pad 1: COL2 -> COL4
- S5 pad 2: c2_r0 -> c4_r0
- S6 pad 1: COL2 -> COL0
- S6 pad 2: c2_r1 -> mirror_c0_r0
- S7 pad 1: COL2 -> COL1
- S7 pad 2: c2_r2 -> mirror_c1_r0
- S8 pad 1: COL3 -> COL2
- S8 pad 2: c3_r0 -> mirror_c2_r0
- S9 pad 2: c3_r1 -> mirror_c3_r0
Other:
- board size 275.6 x 98.2 mm -> 246.6 x 91 mm
