File: pcb/kicad/keyboard.kicad_pcb (KiCad board)
At the start: 2 copper layers, 246.6 x 91 mm, 108 parts

Commit message: pcb: rebuild board (custom outline, 3u half-gap) + hand-place XIAO BLE Plus
Board regenerated from the layout tool with the hand-drawn outline and a
3-unit center-to-center gap between the halves' inner columns, then the
XIAO BLE Plus MCUs placed by hand (footprints embedded in the board, so
the project loads standalone). Adds the KiCad project file.
Parts:
- added U**: XIAO_BLE_Plus, atlas:mcu_xiao_ble_plus, B.Cu at (318.1, -83.5)
- added U**: XIAO_BLE_Plus, atlas:mcu_xiao_ble_plus, B.Cu at (89.5, -83.5)
- moved S19 229.4 mm to (318.1, -46.9)
- moved S6 214.2 mm to (108.6, -77.0)
- moved S20 209.8 mm to (318.1, -65.9)
- moved S21 176.3 mm to (299.1, -38.9)
- moved S7 170.4 mm to (127.6, -41.9)
- moved S15 153.9 mm to (165.7, -75.0)
- moved S22 153.6 mm to (299.1, -57.9)
- moved S8 152.5 mm to (127.6, -61.0)
- moved S9 138.5 mm to (127.6, -80.0)
- moved S16 137.2 mm to (167.1, -16.5), turned to 166 degrees
- moved S23 133.4 mm to (299.1, -77.0)
- moved S29 115.9 mm to (261.0, -77.0)
- moved S17 105.6 mm to (186.2, -10.5), turned to 159 degrees
- moved S10 94.2 mm to (146.7, -38.9)
- moved S32 85.3 mm to (241.9, -75.0), turned to 180 degrees
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Connections:
- S10 pad 1: COL4 -> COL3
- S10 pad 2: mirror_c4_r0 -> c3_r0
- S11 pad 1: COL0 -> COL3
- S11 pad 2: c0_r1 -> c3_r1
- S12 pad 1: COL1 -> COL3
- S12 pad 2: c1_r1 -> c3_r2
- S13 pad 1: COL2 -> COL4
- S13 pad 2: c2_r1 -> c4_r0
- S15 pad 1: COL0 -> COL4
- S15 pad 2: mirror_c0_r1 -> c4_r2
- S16 pad 1: COL1 -> TCOL0
- S16 pad 2: mirror_c1_r1 -> t0_thumb
- S17 pad 1: COL2 -> TCOL1
- S17 pad 2: mirror_c2_r1 -> t1_thumb
- S18 pad 1: COL4 -> COL0
- S18 pad 2: mirror_c4_r1 -> mirror_c0_r0
- S19 pad 2: c0_r2 -> mirror_c0_r1
- S2 pad 1: COL1 -> COL0
- S2 pad 2: c1_r0 -> c0_r1
- S20 pad 1: COL1 -> COL0
- S20 pad 2: c1_r2 -> mirror_c0_r2
- S21 pad 1: COL2 -> COL1
- S21 pad 2: c2_r2 -> mirror_c1_r0
- S22 pad 1: COL3 -> COL1
- S22 pad 2: c3_r2 -> mirror_c1_r1
- S23 pad 1: COL4 -> COL1
- S23 pad 2: c4_r2 -> mirror_c1_r2
- S24 pad 1: COL0 -> COL2
- S24 pad 2: mirror_c0_r2 -> mirror_c2_r0
- S25 pad 1: COL1 -> COL2
- S25 pad 2: mirror_c1_r2 -> mirror_c2_r1
- S27 pad 2: mirror_c3_r2 -> mirror_c3_r0
- S28 pad 1: COL4 -> COL3
- S28 pad 2: mirror_c4_r2 -> mirror_c3_r1
- S29 pad 2: c3_r1 -> mirror_c3_r2
- S3 pad 1: COL2 -> COL0
- S3 pad 2: c2_r0 -> c0_r2
- S30 pad 1: COL3 -> COL4
- S30 pad 2: mirror_c3_r1 -> mirror_c4_r0
- S31 pad 1: TCOL0 -> COL4
- S31 pad 2: t0_thumb -> mirror_c4_r1
- S32 pad 1: TCOL1 -> COL4
- S32 pad 2: t1_thumb -> mirror_c4_r2
- S4 pad 1: COL3 -> COL1
- S4 pad 2: c3_r0 -> c1_r0
- S5 pad 1: COL4 -> COL1
- S5 pad 2: c4_r0 -> c1_r1
- S6 pad 1: COL0 -> COL1
- S6 pad 2: mirror_c0_r0 -> c1_r2
- S7 pad 1: COL1 -> COL2
- S7 pad 2: mirror_c1_r0 -> c2_r0
- S8 pad 2: mirror_c2_r0 -> c2_r1
- S9 pad 1: COL3 -> COL2
- S9 pad 2: mirror_c3_r0 -> c2_r2
Other:
- board size 246.6 x 91 mm -> 247.6 x 96.2 mm
