File: pcb/kicad/keyboard.kicad_pcb (KiCad board)
At the start: 2 copper layers, 247.6 x 96.2 mm, 110 parts

Commit message: pcb: place power switches (Alps SSSS811101) on the board
Hand-placed the SMD side power switch (LCSC C109335) per half, with its
3D model oriented to match the back-side mount.
Parts:
- added SW: PWR_SW, atlas:power_switch_smd_side, F.Cu at (88.6, 96.5)
- added SW: PWR_SW, atlas:power_switch_smd_side, F.Cu at (327.3, 96.5)
- moved D14 189.5 mm to (163.8, 129.5)
- moved D31 189.5 mm to (240.1, 129.5)
- moved LED19 189.5 mm to (322.2, 137.7)
- moved LED2 189.5 mm to (93.7, 137.7)
- moved LED26 189.5 mm to (284.1, 104.6)
- moved LED9 189.5 mm to (131.8, 104.6)
- moved S11 189.5 mm to (150.8, 131.6)
- moved S14 189.5 mm to (169.8, 133.5)
- moved S22 189.5 mm to (303.2, 131.6)
- moved S25 189.5 mm to (284.1, 128.5)
- moved S28 189.5 mm to (265.1, 131.6)
- moved S31 189.5 mm to (246.1, 133.5)
- moved S5 189.5 mm to (112.7, 131.6)
- moved S8 189.5 mm to (131.8, 128.5)
- moved D1 189.5 mm to (87.7, 157.7)
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
Commit message: pcb: fix hotswap socket 3D model depth (offset Z 0 -> 1)
The Kailh hotswap socket STEP (CONN-SMD_HOTPLUGPAKAGE C9900010116) was
attached at Z offset 0, sinking the socket body ~1 mm into the PCB in the
3D view. The model's origin sits ~1.85 mm into +Z, so it needs a +1 mm
push to sit flush against the back copper. Applied to all 34 switch
instances.

KiCad 10 also reserialized the whole file on save; the only geometry
delta is the 34 socket offsets.
Parts:
- SW (x2): moved to B.Cu
- U** (x2): moved to F.Cu

Commit message: pcb: integrate ADS1220 ADC front-end (badjeff reference)
Vendor badjeff/ads1220-pcb (CERN-OHL-P v2) into the board:
- add ads1220.pretty footprint lib (ADS1220 VQFN-16 + 3D model),
  registered in fp-lib-table; bake the .step model path into the
  footprint so it renders without per-instance setup
- append the ADS1220 front-end (U1 + RC network + decoupling) onto
  the board; through-hole breakout headers removed (routes direct
  to XIAO)
- keep badjeff's board + schematic under pcb/kicad/ref/ as the
  net-by-net routing reference
Parts:
- added C1: 0.1uF, Capacitor_SMD:C_0402_1005Metric, B.Cu at (318.7, 104.4)
- added C1: 0.1uF, Capacitor_SMD:C_0402_1005Metric, B.Cu at (89.9, 104.4)
- added C2: 0.1uF, Capacitor_SMD:C_0402_1005Metric, B.Cu at (89.9, 106.2)
- added C2: 0.1uF, Capacitor_SMD:C_0402_1005Metric, B.Cu at (318.7, 106.3)
- added R1: 47R, Resistor_SMD:R_0402_1005Metric, B.Cu at (90.6, 102.5)
- added R1: 47R, Resistor_SMD:R_0402_1005Metric, B.Cu at (319.4, 102.6)
- added R10: 0R, Resistor_SMD:R_0402_1005Metric, B.Cu at (324.6, 108.5)
- added R10: 0R, Resistor_SMD:R_0402_1005Metric, B.Cu at (95.9, 108.5)
- added R11: 0R, Resistor_SMD:R_0402_1005Metric, B.Cu at (97.7, 108.0)
- added R11: 0R, Resistor_SMD:R_0402_1005Metric, B.Cu at (326.5, 108.1)
- added R2: 47R, Resistor_SMD:R_0402_1005Metric, B.Cu at (321.5, 102.6)
- added R2: 47R, Resistor_SMD:R_0402_1005Metric, B.Cu at (92.7, 102.5)
- added R3: 47R, Resistor_SMD:R_0402_1005Metric, B.Cu at (95.1, 102.5)
- added R3: 47R, Resistor_SMD:R_0402_1005Metric, B.Cu at (323.9, 102.6)
- added R4: 47R, Resistor_SMD:R_0402_1005Metric, B.Cu at (326.0, 102.9)
- added R4: 47R, Resistor_SMD:R_0402_1005Metric, B.Cu at (97.2, 102.8)
- added R5: 2K4, Resistor_SMD:R_0402_1005Metric, B.Cu at (326.0, 106.5)
- added R5: 2K4, Resistor_SMD:R_0402_1005Metric, B.Cu at (97.2, 106.4)
- added R6: 2K4, Resistor_SMD:R_0402_1005Metric, B.Cu at (326.0, 104.6)
- added R6: 2K4, Resistor_SMD:R_0402_1005Metric, B.Cu at (97.2, 104.5)
- added R7: 0R, Resistor_SMD:R_0402_1005Metric, B.Cu at (89.4, 108.0)
- added R7: 0R, Resistor_SMD:R_0402_1005Metric, B.Cu at (318.2, 108.1)
- added R8: 0R, Resistor_SMD:R_0402_1005Metric, B.Cu at (91.3, 108.5)
- added R8: 0R, Resistor_SMD:R_0402_1005Metric, B.Cu at (320.1, 108.5)
- added R9: 0R, Resistor_SMD:R_0402_1005Metric, B.Cu at (93.5, 108.5)
- added R9: 0R, Resistor_SMD:R_0402_1005Metric, B.Cu at (322.3, 108.5)
- added U1: ADS1220IRVAR, ads1220:QFN50P350X350X100-17N, B.Cu at (322.0, 105.5)
- added U1: ADS1220IRVAR, ads1220:QFN50P350X350X100-17N, B.Cu at (93.2, 105.4)
Routing:
- net GND: track 0.00 -> 36.7 mm, vias 0 -> 6
- net Net-(R10-Pad1): track 0.00 -> 36.6 mm, vias 0 -> 10
- net REFN0: track 0.00 -> 26.5 mm, vias 0 -> 2
- net REFP0: track 0.00 -> 21.9 mm, vias 0 -> 4
- net DRDY: track 0.00 -> 16.9 mm, vias 0 -> 2
- net 3v3: track 0.00 -> 15.8 mm
- net AIN2: track 0.00 -> 9.84 mm
- net AIN0: track 0.00 -> 9.84 mm
- net AIN1: track 0.00 -> 8.85 mm
- net AIN3: track 0.00 -> 8.53 mm
- net Net-(U1-CS): track 0.00 -> 6.07 mm
- net Net-(U1-DOUT/DRDY): track 0.00 -> 5.64 mm
- net CS: track 0.00 -> 4.54 mm
- net Net-(U1-SCLK): track 0.00 -> 3.81 mm
- net MISO: track 0.00 -> 3.39 mm
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Other:
- rule pad_to_mask_clearance: 0.05 -> 0
- board text added: "3v3"
- board text added: "ADS1220 PCB v1.0 By badjeff"
- board text added: "AIN0"
- board text added: "AIN1"
- board text added: "AIN2"
- board text added: "AIN3"
- board text added: "CS"
- board text added: "DRDY"
- board text added: "GND"
- board text added: "MISO"
- board text added: "MOSI"
- board text added: "REFN0"
- board text added: "REFP0"
- board text added: "SCLK"
