File: pcb/kicad/keyboard.kicad_pcb (KiCad board)
At the start: 2 copper layers, 247.6 x 96.2 mm, 140 parts, among them U1 ADS1220IRVAR

Commit message: pcb: assign matrix + power + ADC nets to both XIAOs
The MCU pads were unconnected (no nets), so routing had no targets.
Assign every XIAO pad its net from the verified pin map (firmware
matrix + Seeed XIAO Plus pinout):
- rows D0-D3, cols D4/D5/D8/D9/D10, 3v3/GND
- ADC SPI on the Plus secondary pins: CS=D11, DRDY=D12, SCLK=D17,
  MISO=D18, MOSI=D19
- thumbs folded into the matrix (TROW0->ROW3, TCOL0/1->COL3/4)
- right half split onto R_-prefixed nets so airwires don't cross the
  BT split; right columns mirrored (reversed) per the firmware
Verified: 16 nets per XIAO, no net crosses the L/R split, file loads
clean in kicad-cli.
Connections:
- net led_din_mirror_matrix_c0_r0 renamed R_led_din_mirror_matrix_c0_r0
- net led_din_mirror_matrix_c0_r1 renamed R_led_din_mirror_matrix_c0_r1
- net led_din_mirror_matrix_c0_r2 renamed R_led_din_mirror_matrix_c0_r2
- net led_din_mirror_matrix_c1_r0 renamed R_led_din_mirror_matrix_c1_r0
- net led_din_mirror_matrix_c1_r1 renamed R_led_din_mirror_matrix_c1_r1
- net led_din_mirror_matrix_c1_r2 renamed R_led_din_mirror_matrix_c1_r2
- net led_din_mirror_matrix_c2_r0 renamed R_led_din_mirror_matrix_c2_r0
- net led_din_mirror_matrix_c2_r1 renamed R_led_din_mirror_matrix_c2_r1
- net led_din_mirror_matrix_c2_r2 renamed R_led_din_mirror_matrix_c2_r2
- net led_din_mirror_matrix_c3_r0 renamed R_led_din_mirror_matrix_c3_r0
- net led_din_mirror_matrix_c3_r1 renamed R_led_din_mirror_matrix_c3_r1
- net led_din_mirror_matrix_c3_r2 renamed R_led_din_mirror_matrix_c3_r2
- net led_din_mirror_matrix_c4_r0 renamed R_led_din_mirror_matrix_c4_r0
- net led_din_mirror_matrix_c4_r1 renamed R_led_din_mirror_matrix_c4_r1
- net led_din_mirror_matrix_c4_r2 renamed R_led_din_mirror_matrix_c4_r2
- net led_din_mirror_thumbs_t0_thumb renamed R_led_din_mirror_thumbs_t0_thumb
- net led_din_mirror_thumbs_t1_thumb renamed R_led_din_mirror_thumbs_t1_thumb
- net led_dout_mirror_matrix_c0_r0 renamed R_led_dout_mirror_matrix_c0_r0
- net led_dout_mirror_matrix_c0_r1 renamed R_led_dout_mirror_matrix_c0_r1
- net led_dout_mirror_matrix_c0_r2 renamed R_led_dout_mirror_matrix_c0_r2
- net led_dout_mirror_matrix_c1_r0 renamed R_led_dout_mirror_matrix_c1_r0
- net led_dout_mirror_matrix_c1_r1 renamed R_led_dout_mirror_matrix_c1_r1
- net led_dout_mirror_matrix_c1_r2 renamed R_led_dout_mirror_matrix_c1_r2
- net led_dout_mirror_matrix_c2_r0 renamed R_led_dout_mirror_matrix_c2_r0
- net led_dout_mirror_matrix_c2_r1 renamed R_led_dout_mirror_matrix_c2_r1
- net led_dout_mirror_matrix_c2_r2 renamed R_led_dout_mirror_matrix_c2_r2
- net led_dout_mirror_matrix_c3_r0 renamed R_led_dout_mirror_matrix_c3_r0
- net led_dout_mirror_matrix_c3_r1 renamed R_led_dout_mirror_matrix_c3_r1
- net led_dout_mirror_matrix_c3_r2 renamed R_led_dout_mirror_matrix_c3_r2
- net led_dout_mirror_matrix_c4_r0 renamed R_led_dout_mirror_matrix_c4_r0
- net led_dout_mirror_matrix_c4_r1 renamed R_led_dout_mirror_matrix_c4_r1
- net led_dout_mirror_matrix_c4_r2 renamed R_led_dout_mirror_matrix_c4_r2
- net led_dout_mirror_thumbs_t0_thumb renamed R_led_dout_mirror_thumbs_t0_thumb
- net led_dout_mirror_thumbs_t1_thumb renamed R_led_dout_mirror_thumbs_t1_thumb
- net mirror_c0_r0 renamed R_mirror_c0_r0
- net mirror_c0_r1 renamed R_mirror_c0_r1
- net mirror_c0_r2 renamed R_mirror_c0_r2
- net mirror_c1_r0 renamed R_mirror_c1_r0
- net mirror_c1_r1 renamed R_mirror_c1_r1
- net mirror_c1_r2 renamed R_mirror_c1_r2
- net mirror_c2_r0 renamed R_mirror_c2_r0
- net mirror_c2_r1 renamed R_mirror_c2_r1
- net mirror_c2_r2 renamed R_mirror_c2_r2
- net mirror_c3_r0 renamed R_mirror_c3_r0
- net mirror_c3_r1 renamed R_mirror_c3_r1
- net mirror_c3_r2 renamed R_mirror_c3_r2
- net mirror_c4_r0 renamed R_mirror_c4_r0
- net mirror_c4_r1 renamed R_mirror_c4_r1
- net mirror_c4_r2 renamed R_mirror_c4_r2
- net mirror_t0_thumb renamed R_mirror_t0_thumb
- net mirror_t1_thumb renamed R_mirror_t1_thumb
- C1 pad 1: 3v3 -> R_3v3
- C1 pad 2: GND -> R_GND
- C2 pad 1: 3v3 -> R_3v3
- C2 pad 2: GND -> R_GND
- D16 pad 1: TROW0 -> ROW3
- D17 pad 1: TROW0 -> ROW3
- D18 pad 1: ROW0 -> R_ROW0
- D19 pad 1: ROW1 -> R_ROW1
- D20 pad 1: ROW2 -> R_ROW2
- D21 pad 1: ROW0 -> R_ROW0
- D22 pad 1: ROW1 -> R_ROW1
- D23 pad 1: ROW2 -> R_ROW2
- D24 pad 1: ROW0 -> R_ROW0
- D25 pad 1: ROW1 -> R_ROW1
- D26 pad 1: ROW2 -> R_ROW2
- D27 pad 1: ROW0 -> R_ROW0
- D28 pad 1: ROW1 -> R_ROW1
- D29 pad 1: ROW2 -> R_ROW2
- D30 pad 1: ROW0 -> R_ROW0
- D31 pad 1: ROW1 -> R_ROW1
- D32 pad 1: ROW2 -> R_ROW2
- D33 pad 1: TROW0 -> R_ROW3
- D34 pad 1: TROW0 -> R_ROW3
- LED18 pad 1: VCC -> R_VCC
- LED18 pad 3: GND -> R_GND
- LED19 pad 1: VCC -> R_VCC
- LED19 pad 3: GND -> R_GND
- LED20 pad 1: VCC -> R_VCC
- LED20 pad 3: GND -> R_GND
- LED21 pad 1: VCC -> R_VCC
- LED21 pad 3: GND -> R_GND
- LED22 pad 1: VCC -> R_VCC
- LED22 pad 3: GND -> R_GND
- LED23 pad 1: VCC -> R_VCC
- LED23 pad 3: GND -> R_GND
- LED24 pad 1: VCC -> R_VCC
- LED24 pad 3: GND -> R_GND
- LED25 pad 1: VCC -> R_VCC
- LED25 pad 3: GND -> R_GND
- LED26 pad 1: VCC -> R_VCC
- LED26 pad 3: GND -> R_GND
- LED27 pad 1: VCC -> R_VCC
- LED27 pad 3: GND -> R_GND
- LED28 pad 1: VCC -> R_VCC
- LED28 pad 3: GND -> R_GND
- LED29 pad 1: VCC -> R_VCC
- LED29 pad 3: GND -> R_GND
- LED30 pad 1: VCC -> R_VCC
- LED30 pad 3: GND -> R_GND
- LED31 pad 1: VCC -> R_VCC
- LED31 pad 3: GND -> R_GND
- LED32 pad 1: VCC -> R_VCC
- LED32 pad 3: GND -> R_GND
- LED33 pad 1: VCC -> R_VCC
- LED33 pad 3: GND -> R_GND
- LED34 pad 1: VCC -> R_VCC
- LED34 pad 3: GND -> R_GND
- R1 pad 1: Net-(U1-DOUT/DRDY) -> R_Net-(U1-DOUT/DRDY)
- R1 pad 2: MISO -> R_MISO
- R10 pad 1: Net-(R10-Pad1) -> R_Net-(R10-Pad1)
- R10 pad 2: AIN3 -> R_AIN3
- R11 pad 1: REFN0 -> R_REFN0
- R11 pad 2: GND -> R_GND
- R2 pad 1: Net-(U1-DIN) -> R_Net-(U1-DIN)
- R2 pad 2: MOSI -> R_MOSI
- R3 pad 1: Net-(U1-SCLK) -> R_Net-(U1-SCLK)
- R3 pad 2: SCLK -> R_SCLK
- R4 pad 1: Net-(U1-CS) -> R_Net-(U1-CS)
- R4 pad 2: CS -> R_CS
- R5 pad 1: REFP0 -> R_REFP0
- R5 pad 2: Net-(R10-Pad1) -> R_Net-(R10-Pad1)
- R6 pad 1: Net-(R10-Pad1) -> R_Net-(R10-Pad1)
- R6 pad 2: REFN0 -> R_REFN0
- R7 pad 1: Net-(R10-Pad1) -> R_Net-(R10-Pad1)
- R7 pad 2: AIN0 -> R_AIN0
- R8 pad 1: Net-(R10-Pad1) -> R_Net-(R10-Pad1)
- R8 pad 2: AIN1 -> R_AIN1
- R9 pad 1: Net-(R10-Pad1) -> R_Net-(R10-Pad1)
- R9 pad 2: AIN2 -> R_AIN2
- S16 pad 1: TCOL0 -> COL3
- S17 pad 1: TCOL1 -> COL4
- S18 pad 1: COL0 -> R_COL0
- S19 pad 1: COL0 -> R_COL0
- S20 pad 1: COL0 -> R_COL0
- S21 pad 1: COL1 -> R_COL1
- S22 pad 1: COL1 -> R_COL1
- S23 pad 1: COL1 -> R_COL1
- S24 pad 1: COL2 -> R_COL2
- S25 pad 1: COL2 -> R_COL2
- S26 pad 1: COL2 -> R_COL2
- S27 pad 1: COL3 -> R_COL3
- S28 pad 1: COL3 -> R_COL3
- S29 pad 1: COL3 -> R_COL3
- S30 pad 1: COL4 -> R_COL4
- S31 pad 1: COL4 -> R_COL4
- S32 pad 1: COL4 -> R_COL4
- S33 pad 1: TCOL0 -> R_COL3
- S34 pad 1: TCOL1 -> R_COL4
- U** pad 1: (no net) -> R_ROW0
- U** pad 10: (no net) -> R_COL1
- U** pad 11: (no net) -> R_COL2
- U** pad 12: (no net) -> R_3v3
- U** pad 13: (no net) -> R_GND
- U** pad 15: (no net) -> R_CS
- U** pad 16: (no net) -> R_DRDY
- U** pad 2: (no net) -> R_ROW1
- U** pad 21: (no net) -> R_SCLK
- U** pad 22: (no net) -> R_MISO
- U** pad 23: (no net) -> R_MOSI
- U** pad 3: (no net) -> R_ROW2
- U** pad 4: (no net) -> R_ROW3
- U** pad 5: (no net) -> R_COL4
- U** pad 6: (no net) -> R_COL3
- U** pad 9: (no net) -> R_COL0
- U** pad 1: (no net) -> ROW0
- U** pad 10: (no net) -> COL3
- U** pad 11: (no net) -> COL2
- U** pad 12: (no net) -> 3v3
- U** pad 13: (no net) -> GND
- U** pad 15: (no net) -> CS
- U** pad 16: (no net) -> DRDY
- U** pad 2: (no net) -> ROW1
- U** pad 21: (no net) -> SCLK
- U** pad 22: (no net) -> MISO
- U** pad 23: (no net) -> MOSI
- U** pad 3: (no net) -> ROW2
- U** pad 4: (no net) -> ROW3
- U** pad 5: (no net) -> COL0
- U** pad 6: (no net) -> COL1
- U** pad 9: (no net) -> COL4
- U1 pad 1: GND -> R_GND
- U1 pad 10: 3v3 -> R_3v3
- U1 pad 11: 3v3 -> R_3v3
- U1 pad 12: DRDY -> R_DRDY
- U1 pad 13: Net-(U1-DOUT/DRDY) -> R_Net-(U1-DOUT/DRDY)
- U1 pad 14: Net-(U1-DIN) -> R_Net-(U1-DIN)
- U1 pad 15: Net-(U1-SCLK) -> R_Net-(U1-SCLK)
- U1 pad 16: Net-(U1-CS) -> R_Net-(U1-CS)
- U1 pad 2: GND -> R_GND
- U1 pad 3: GND -> R_GND
- U1 pad 4: AIN3 -> R_AIN3
- U1 pad 5: AIN2 -> R_AIN2
- U1 pad 6: REFN0 -> R_REFN0
- U1 pad 7: REFP0 -> R_REFP0
- U1 pad 8: AIN1 -> R_AIN1
- U1 pad 9: AIN0 -> R_AIN0

Commit message: pcb: fix reversed right-half column mapping
Verified against switch x-positions: both halves wire pinky=COL0=D4
and inner=COL4=D8 physically (the firmware's left/right col-gpios
reversal is logical numbering only). Right XIAO columns now map
identically to left (pad5->R_COL0 .. pad9->R_COL4), not mirrored.
Connections:
- U** pad 10: R_COL1 -> R_COL3
- U** pad 5: R_COL4 -> R_COL0
- U** pad 6: R_COL3 -> R_COL1
- U** pad 9: R_COL0 -> R_COL4
Changed lines of the file:
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@@
 			(size 2.032 0.95)
 			(layers "F.Cu" "F.Mask" "F.Paste")
-			(net "R_COL4")
+			(net "R_COL0")
 			(roundrect_rratio 0.1)
 		)
@@
 			(size 2.032 0.95)
 			(layers "F.Cu" "F.Mask" "F.Paste")
-			(net "R_COL3")
+			(net "R_COL1")
 			(roundrect_rratio 0.1)
 		)
@@
 			(size 2.032 0.95)
 			(layers "F.Cu" "F.Mask" "F.Paste")
-			(net "R_COL0")
+			(net "R_COL4")
 			(roundrect_rratio 0.1)
 		)
@@
 			(size 2.032 0.95)
 			(layers "F.Cu" "F.Mask" "F.Paste")
-			(net "R_COL1")
+			(net "R_COL3")
 			(roundrect_rratio 0.1)
 		)
